File: pcb/the-zapfish.kicad_sch (KiCad schematic)
At the start: 8 parts, among them J2 Conn_01x02, J3 Conn_01x02, U1 LM317

Commit message: edit
Parts:
- RV1: value 50k -> 5k
Changed lines of the file:
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@@
 			)
 		)
-		(property "Value" "50k"
+		(property "Value" "5k"
 			(at 189.23 114.2999 0)
 			(effects
